File: RPi_Expansion_Board/V2.0/RPi_GPIO.sch (KiCad schematic (older format))
At the start: 21 parts, among them J1 RPi_GPIO, P1 CONN_02X20

Commit message: cambios RPI board
Parts:
- added P2: 5Vcc_, Pin_Headers:Pin_Header_Angled_1x02_Pitch2.54mm, symbol CONN_01X02
Connections:
- wire segments 27 -> 31
Changed lines of the file:
@@
+	1    0    0    -1
+$EndComp
+$Comp
+L CONN_01X04 C1
+U 1 1 58CD3F00
+P 2200 6200
+F 0 "C1" H 2200 6450 50  0000 C CNN
+F 1 " " V 2300 6200 50  0000 C CNN
+F 2 "Pin_Headers:Pin_Header_Straight_1x04_Pitch2.54mm" H 2200 6200 50  0001 C CNN
+F 3 "" H 2200 6200 50  0000 C CNN
+	1    2200 6200
+	-1   0    0    1
+$EndComp
+$Comp
+L CONN_01X04 C2
+U 1 1 58CD4334
+P 2650 6200
+F 0 "C2" H 2650 6450 50  0000 C CNN
+F 1 " " V 2750 6200 50  0000 C CNN
+F 2 "Pin_Headers:Pin_Header_Straight_1x04_Pitch2.54mm" H 2650 6200 50  0001 C CNN
+F 3 "" H 2650 6200 50  0000 C CNN
+	1    2650 6200
+	-1   0    0    1
+$EndComp
+$Comp
+L CONN_01X04 C3
+U 1 1 58CD4381
+P 3100 6200
+F 0 "C3" H 3100 6450 50  0000 C CNN
+F 1 " " V 3200 6200 50  0000 C CNN
+F 2 "Pin_Headers:Pin_Header_Straight_1x04_Pitch2.54mm" H 3100 6200 50  0001 C CNN
+F 3 "" H 3100 6200 50  0000 C CNN
+	1    3100 6200
+	-1   0    0    1
+$EndComp
+$Comp
+L CONN_01X04 C4
+U 1 1 58CD43D5
+P 3500 6200
+F 0 "C4" H 3500 6450 50  0000 C CNN
+F 1 " " V 3600 6200 50  0000 C CNN
+F 2 "Pin_Headers:Pin_Header_Straight_1x04_Pitch2.54mm" H 3500 6200 50  0001 C CNN
+F 3 "" H 3500 6200 50  0000 C CNN
+	1    3500 6200
+	-1   0    0    1
+$EndComp
+$Comp
+L GND #PWR020
+U 1 1 58CD8EDD
+P 800 3000
+F 0 "#PWR020" H 800 2750 50  0001 C CNN
+F 1 "GND" H 800 2850 50  0000 C CNN
+F 2 "" H 800 3000 50  0000 C CNN
+F 3 "" H 800 3000 50  0000 C CNN
+	1    800  3000
+	1    0    0    -1
+$EndComp
+$Comp
+L CONN_01X04 GND2
+U 1 1 58CD8EE3
+P 1000 2750
+F 0 "GND2" H 1000 3000 50  0000 C CNN
+F 1 "GND" V 1100 2750 50  0000 C CNN
+F 2 "Pin_Headers:Pin_Header_Straight_1x04_Pitch2.54mm" H 1000 2750 50  0001 C CNN
+F 3 "" H 1000 2750 50  0000 C CNN
+	1    1000 2750
+	1    0    0    -1
+$EndComp
+$Comp
+L CONN_01X04 C9
+U 1 1 58D1327A
+P 3950 6200
+F 0 "C9" H 3950 6450 50  0000 C CNN
+F 1 " " V 4050 6200 50  0000 C CNN
+F 2 "Pin_Headers:Pin_Header_Straight_1x04_Pitch2.54mm" H 3950 6200 50  0001 C CNN
+F 3 "" H 3950 6200 50  0000 C CNN
+	1    3950 6200
+	-1   0    0    1
+$EndComp
+$Comp
+L CONN_02X20 P1
+U 1 1 58D278FE
+P 2800 3650
+F 0 "P1" H 2800 4700 50  0000 C CNN
+F 1 "CONN_02X20" V 2800 3650 50  0000 C CNN
+F 2 "Pin_Headers:Pin_Header_Straight_2x20_Pitch2.54mm" H 2800 2300 50  0000 C CNN
+F 3 "" H 2800 2700 50  0000 C CNN
+	1    2800 3650
+	-1   0    0    -1
+$EndComp
+$Comp
+L GND #PWR021
+U 1 1 58D2D4B1
+P 1350 6500
+F 0 "#PWR021" H 1350 6250 50  0001 C CNN
+F 1 "GND" H 1350 6350 50  0000 C CNN
+F 2 "" H 1350 6500 50  0000 C CNN
+F 3 "" H 1350 6500 50  0000 C CNN
+	1    1350 6500
+	1    0    0    -1
+$EndComp
+$Comp
+L GND #PWR022
+U 1 1 58D2D99A
+P 1300 7300
+F 0 "#PWR022" H 1300 7050 50  0001 C CNN
+F 1 "GND" H 1300 7150 50  0000 C CNN
+F 2 "" H 1300 7300 50  0000 C CNN
+F 3 "" H 1300 7300 50  0000 C CNN
+	1    1300 7300
+	1    0    0    -1
+$EndComp
+$Comp
+L RPi_GPIO J1
+U 1 1 5515D39E
+P 4700 2750
+F 0 "J1" H 5450 3000 60  0000 C CNN
+F 1 "RPi_GPIO" H 5450 2900 60  0000 C CNN
+F 2 "" H 4700 2750 60  0001 C CNN
+F 3 "" H 4700 2750 60  0000 C CNN
+	1    4700 2750
+	1    0    0    -1
+$EndComp
+$Comp
+L CONN_01X02 P2
+U 1 1 5909301A
+P 7200 1900
+F 0 "P2" H 7200 2050 50  0000 C CNN
+F 1 "5Vcc_" V 7300 1900 50  0000 C CNN
+F 2 "Pin_Headers:Pin_Header_Angled_1x02_Pitch2.54mm" H 7200 1900 50  0001 C CNN
+F 3 "" H 7200 1900 50  0000 C CNN
+	1    7200 1900
+	1    0    0    -1
+$EndComp
+$Comp
+L GND #PWR023
+U 1 1 590930FB
+P 6900 2000
+F 0 "#PWR023" H 6900 1750 50  0001 C CNN
+F 1 "GND" H 6900 1850 50  0000 C CNN
+F 2 "" H 6900 2000 50  0000 C CNN
+F 3 "" H 6900 2000 50  0000 C CNN
+	1    6900 2000
+	1    0    0    -1
+$EndComp
+$Comp
+L +5V #PWR024
+U 1 1 59093148
+P 6900 1800
+F 0 "#PWR024" H 6900 1650 50  0001 C CNN
+F 1 "+5V" H 6900 1940 50  0000 C CNN
+F 2 "" H 6900 1800 50  0000 C CNN
+F 3 "" H 6900 1800 50  0000 C CNN
+	1    6900 1800
 	1    0    0    -1
 $EndComp
@@
 Wire Wire Line
 	2150 800  2150 1300
-$Comp
-L CONN_01X04 C1
-U 1 1 58CD3F00
-P 2200 6200
-F 0 "C1" H 2200 6450 50  0000 C CNN
-F 1 " " V 2300 6200 50  0000 C CNN
-F 2 "Pin_Headers:Pin_Header_Straight_1x04_Pitch2.54mm" H 2200 6200 50  0001 C CNN
-F 3 "" H 2200 6200 50  0000 C CNN
-	1    2200 6200
-	-1   0    0    1
-$EndComp
-$Comp
-L CONN_01X04 C2
-U 1 1 58CD4334
-P 2650 6200
-F 0 "C2" H 2650 6450 50  0000 C CNN
-F 1 " " V 2750 6200 50  0000 C CNN
-F 2 "Pin_Headers:Pin_Header_Straight_1x04_Pitch2.54mm" H 2650 6200 50  0001 C CNN
-F 3 "" H 2650 6200 50  0000 C CNN
-	1    2650 6200
-	-1   0    0    1
-$EndComp
-$Comp
-L CONN_01X04 C3
-U 1 1 58CD4381
-P 3100 6200
-F 0 "C3" H 3100 6450 50  0000 C CNN
-F 1 " " V 3200 6200 50  0000 C CNN
-F 2 "Pin_Headers:Pin_Header_Straight_1x04_Pitch2.54mm" H 3100 6200 50  0001 C CNN
-F 3 "" H 3100 6200 50  0000 C CNN
-	1    3100 6200
-	-1   0    0    1
-$EndComp
-$Comp
-L CONN_01X04 C4
-U 1 1 58CD43D5
-P 3500 6200
-F 0 "C4" H 3500 6450 50  0000 C CNN
-F 1 " " V 3600 6200 50  0000 C CNN
-F 2 "Pin_Headers:Pin_Header_Straight_1x04_Pitch2.54mm" H 3500 6200 50  0001 C CNN
-F 3 "" H 3500 6200 50  0000 C CNN
-	1    3500 6200
-	-1   0    0    1
-$EndComp
 Wire Wire Line
 	3700 6050 3700 6350
@@
 Connection ~ 3700 6250
 Connection ~ 3700 6150
-$Comp
-L GND #PWR020
-U 1 1 58CD8EDD
-P 800 3000
-F 0 "#PWR020" H 800 2750 50  0001 C CNN
-F 1 "GND" H 800 2850 50  0000 C CNN
-F 2 "" H 800 3000 50  0000 C CNN
-F 3 "" H 800 3000 50  0000 C CNN
-	1    800  3000
-	1    0    0    -1
-$EndComp
-$Comp
-L CONN_01X04 GND2
-U 1 1 58CD8EE3
-P 1000 2750
-F 0 "GND2" H 1000 3000 50  0000 C CNN
-F 1 "GND" V 1100 2750 50  0000 C CNN
-F 2 "Pin_Headers:Pin_Header_Straight_1x04_Pitch2.54mm" H 1000 2750 50  0001 C CNN
-F 3 "" H 1000 2750 50  0000 C CNN
-	1    1000 2750
-	1    0    0    -1
-$EndComp
 Connection ~ 800  2800
 Connection ~ 800  2900
@@
 Wire Wire Line
 	800  2500 800  3000
-$Comp
-L CONN_01X04 C9
-U 1 1 58D1327A
-P 3950 6200
-F 0 "C9" H 3950 6450 50  0000 C CNN
-F 1 " " V 4050 6200 50  0000 C CNN
-F 2 "Pin_Headers:Pin_Header_Straight_1x04_Pitch2.54mm" H 3950 6200 50  0001 C CNN
-F 3 "" H 3950 6200 50  0000 C CNN
-	1    3950 6200
-	-1   0    0    1
-$EndComp
 Wire Wire Line
 	4150 6050 4150 6350
 Connection ~ 4150 6250
 Connection ~ 4150 6150
-$Comp
-L CONN_02X20 P1
-U 1 1 58D278FE
-P 2800 3650
-F 0 "P1" H 2800 4700 50  0000 C CNN
-F 1 "CONN_02X20" V 2800 3650 50  0000 C CNN
-F 2 "Pin_Headers:Pin_Header_Straight_2x20_Pitch2.54mm" H 2800 2300 50  0000 C CNN
-F 3 "" H 2800 2700 50  0000 C CNN
-	1    2800 3650
-	-1   0    0    -1
-$EndComp
 Connection ~ 1900 4600
 Wire Wire Line
 	2550 3300 2500 3300
-$Comp
-L GND #PWR021
-U 1 1 58D2D4B1
-P 1350 6500
-F 0 "#PWR021" H 1350 6250 50  0001 C CNN
-F 1 "GND" H 1350 6350 50  0000 C CNN
-F 2 "" H 1350 6500 50  0000 C CNN
-F 3 "" H 1350 6500 50  0000 C CNN
-	1    1350 6500
-	1    0    0    -1
-$EndComp
 Connection ~ 1350 6300
 Connection ~ 1350 6400
@@
 Wire Wire Line
 	1350 6000 1350 6500
-$Comp
-L GND #PWR022
-U 1 1 58D2D99A
-P 1300 7300
-F 0 "#PWR022" H 1300 7050 50  0001 C CNN
-F 1 "GND" H 1300 7150 50  0000 C CNN
-F 2 "" H 1300 7300 50  0000 C CNN
-F 3 "" H 1300 7300 50  0000 C CNN
-	1    1300 7300
-	1    0    0    -1
-$EndComp
 Connection ~ 1300 7100
 Connection ~ 1300 7200
@@
 Wire Wire Line
 	1300 6800 1300 7300
-$Comp
-L RPi_GPIO J1
-U 1 1 5515D39E
-P 4700 2750
-F 0 "J1" H 5450 3000 60  0000 C CNN
-F 1 "RPi_GPIO" H 5450 2900 60  0000 C CNN
-F 2 "" H 4700 2750 60  0001 C CNN
-F 3 "" H 4700 2750 60  0000 C CNN
-	1    4700 2750
-	1    0    0    -1
-$EndComp
 Wire Wire Line
 	2400 6050 3300 6050
@@
 	2400 6350 3300 6350
 Connection ~ 2850 6350
+Wire Wire Line
+	7000 1850 6900 1850
+Wire Wire Line
+	6900 1850 6900 1800
+Wire Wire Line
+	7000 1950 6900 1950
+Wire Wire Line
+	6900 1950 6900 2000
 $EndSCHEMATC
