File: RPi_Expansion_Board/V2.0/RPi_Hat_k3.kicad_pcb (KiCad board)
At the start: 2 copper layers, 65 x 56.5 mm, 23 parts, among them P1 CONN_02X20

Commit message: include logos
Parts:
- added G***: LOGO, RpiHat:creatvra, F.Cu at (97.5, 78.6)
- added G***: LOGO, RpiHat:openHW, F.Cu at (153.4, 86.9)
- added G***: LOGO, RpiHat:ECCI, F.Cu at (98.2, 109.1)

Commit message: cambios en la board de expansion RPI
Parts:
- added P2: power5vcc, Pin_Headers:Pin_Header_Angled_1x02_Pitch2.54mm, B.Cu at (100.7, 78.6)
- moved G*** 2.29 mm to (95.6, 79.9)
Routing:
- net GND: track 278.3 -> 283.3 mm
- net +5V: track 131.6 -> 136.0 mm
- added copper zone on B.Cu, net GND
- added copper zone on F.Cu, net GND

Commit message: Cambios de la PCB
Parts:
- moved G*** 0.80 mm to (96.4, 80.2)
- renumbered P2 to 5V
