File: RPi_Expansion_Board/V2.0/RPi_Hat_k3.kicad_pcb (KiCad board)
At the start: 2 copper layers, 65 x 56.5 mm, 27 parts, among them P1 CONN_02X20, P2 power5vcc

Commit message: cambios en la RPI expansion board y logos
Parts:
- moved G*** 30.6 mm to (98.8, 110.4)
- moved G*** 15.3 mm to (99.4, 93.9)
